File: nautilus/hw/nautilus.kicad_sch (KiCad schematic)
At the start: 100 parts, among them IC1 DRV8353SRTAR, IC2 STM32G474CEU6, IC3 MAX15062AATA+T, J1 XT30XT30PW_MALE, J2 Conn_01x02_Pin, J3 Conn_01x02_Pin, U2 CSD88599Q5DCT, U3 CSD88599Q5DCT, U4 AS5147, U5 CSD88599Q5DCT

Commit message: First PCB layout, before DRC.
Parts:
- removed ENC1: PICO-SPOX-6NOPASTE, Connector_JST:JST_SH_SM06B-SRSS-TB_1x06-1MP_P1.00mm_Horizontal, symbol nautilus-eagle-import:PICO-SPOX-6NOPASTE
- added C50, C51: 10nF, Capacitor_SMD:C_0402_1005Metric_Pad0.74x0.62mm_HandSolder, symbol Device:C
- added C52: 0.1uF, Capacitor_SMD:C_0402_1005Metric_Pad0.74x0.62mm_HandSolder, symbol Device:C
- added JP1: SolderJumper_2_Bridged, Jumper:SolderJumper-2_P1.3mm_Bridged2Bar_Pad1.0x1.5mm, symbol Jumper:SolderJumper_2_Bridged
- added R19, R20: 5k, Resistor_SMD:R_0402_1005Metric_Pad0.72x0.64mm_HandSolder, symbol Device:R
- added R21: 100k, Resistor_SMD:R_0402_1005Metric_Pad0.72x0.64mm_HandSolder, symbol Device:R
- added SPI2: JST_SH4, Connector_JST:JST_SH_SM04B-SRSS-TB_1x04-1MP_P1.00mm_Horizontal, symbol nautilus-eagle-import:JST_ZH4
- C27: value 1uF 100V -> 1uF; footprint Capacitor_SMD:C_0805_2012Metric_Pad1.18x1.45mm_HandSolder -> Capacitor_SMD:C_0603_1608Metric_Pad1.08x0.95mm_HandSolder; HOUSEPART (none) -> 1; MF MURATA -> (none); MPN GCM21BC72A105KE36L -> MF-CAP-0603-1uF
- C33: value 0.01uF -> 10nF
- C44: footprint Capacitor_SMD:C_1206_3216Metric_Pad1.33x1.80mm_HandSolder -> Capacitor_SMD:C_0402_1005Metric_Pad0.74x0.62mm_HandSolder; HOUSEPART 1 -> YES; MPN MF-CAP-1206-10uF -> MF-CAP-0402-1uF
- C5: footprint Capacitor_SMD:C_0603_1608Metric_Pad1.08x0.95mm_HandSolder -> Capacitor_SMD:C_0402_1005Metric_Pad0.74x0.62mm_HandSolder; MF TDK -> (none); MPN C1608X7R1E105K080AE -> MF-CAP-0402-1uF
- H2: footprint MountingHole:MountingHole_2.2mm_M2_ISO7380 -> MountingHole:MountingHole_2.2mm_M2_ISO7380_Pad; symbol Mechanical:MountingHole -> Mechanical:MountingHole_Pad
- R1: value 2k -> 10k
- RA1, RA2, RA3: value 0.5mOhm 1% 2W -> 1.0mOhm 1% 2W
- SPI1: value JST_ZH4 -> JST_ZH5; footprint Connector_JST:JST_SH_SM04B-SRSS-TB_1x04-1MP_P1.00mm_Horizontal -> Connector_JST:JST_GH_SM05B-GHS-TB_1x05-1MP_P1.25mm_Horizontal; symbol nautilus-eagle-import:JST_ZH4 -> Connector_Generic:Conn_01x05
- renumbered MOT1 to M1, MOT2 to M2, MOT3 to M3
Connections:
- net SECONDARY_ENC_CS is gone; now on net MOTOR_HIZ: IC2.2 (PC13)
- net DEBUG1: now also IC2.34 (PA12); no longer IC2.3 (PC14-OSC32_IN)
- net DEBUG2: now also IC2.33 (PA11); no longer IC2.4 (PC15-OSC32_OUT)
- net DRV8323_CS: now also IC2.4 (PC15-OSC32_OUT); no longer IC2.29 (PC6)
- net LED1: now also IC2.44 (PB6); no longer IC2.5 (PF0-OSC_IN)
- net LED2: now also IC2.45 (PB7); no longer IC2.6 (PF1-OSC_OUT)
- net MOTOR_FAULT: now also IC2.3 (PC14-OSC32_IN); no longer IC2.44 (PB6)
- net MOTOR_HIZ: no longer IC2.45 (PB7)
- net SXB_P: now also RA2.2; no longer RA3.2
- net SXC_P: now also RA3.2; no longer RA2.2
- net VTEMP_MOT: now also C50.1
- net at IC1.40 (VGLS): now also C5.1; no longer C5.2
- net I2C_ABS_SCL: now reaches IC2.46 (PB8-BOOT0)
- net I2C_ABS_SCL: now also R19.2, SPI2.4
- net I2C_ABS_SDA: now reaches IC2.47 (PB9)
- net I2C_ABS_SDA: now also R20.2, SPI2.3
- net +3V3 renamed +3.3V
- net +3.3V: now also C52.1, R19.1, R20.1, SPI2.2
- net GND renamed GNDS
- net GNDS: now also SPI1.5 (Pin_5), C50.2, C52.2, JP1.2 (B), SPI2.1; no longer C1.2, C17.2, C25.2, C28.2, C29.2, C3.2, C31.2, C32.2, C34.2, C35.2, C36.2, C37.2, C38.2, C39.2, C40.2, C41.2, C42.2, C43.2, C45.2, C47.2, C5.1, C8.2, IC1.10 (SNA), IC1.11 (SNB), IC1.20 (SNC), IC1.39 (GND), J1.2, RA1.1, RA2.1, RA3.1
- new net: C51.1, H2.1, R21.1
- new net GNDPWR: C1.2, C17.2, C25.2, C28.2, C29.2, C3.2, C31.2, C32.2, C34.2, C35.2, C36.2, C37.2, C38.2, C39.2, C40.2, C41.2, C42.2, C43.2, C45.2, C47.2, C5.2, C51.2, C8.2, IC1.10 (SNA), IC1.11 (SNB), IC1.20 (SNC), IC1.39 (GND), J1.2, JP1.1 (A), R21.2, RA1.1, RA2.1, RA3.1
Other:
- note added: "Why is this to GNDS and not PWR GND ?"
- note added: "nautilus v1.0"
- note removed: "moteus r4.11 (c) jjp@pobox.com 2022 Licensed under the Apache 2.0 License"
- moved on the sheet: C10, C11, C12, C14, C15, C16, C17, C18, C19, C20, C21, C23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

Commit message: First PCB design passing DRC
Parts:
- H2: footprint MountingHole:MountingHole_2.2mm_M2_ISO7380_Pad -> nautilus:MountingHole-Plated
Changed lines of the file:
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@@
       (effects (font (size 1.27 1.27)) (justify left))
     )
-    (property "Footprint" "MountingHole:MountingHole_2.2mm_M2_ISO7380_Pad" (at 46.99 139.7 0)
+    (property "Footprint" "nautilus:MountingHole-Plated" (at 46.99 139.7 0)
       (effects (font (size 1.27 1.27)) hide)
     )

Commit message: Cleanup PCB before order
Parts:
- removed JP1: SolderJumper_2_Bridged, Jumper:SolderJumper-2_P1.3mm_Bridged2Bar_Pad1.0x1.5mm, symbol Jumper:SolderJumper_2_Bridged
- added C53: 10uF 50V, Capacitor_SMD:C_1206_3216Metric_Pad1.33x1.80mm_HandSolder, symbol Device:C
- added C54, C55, C56, C57: 10uF, Capacitor_SMD:C_1206_3216Metric_Pad1.33x1.80mm_HandSolder, symbol Device:C
- added D3, D4: D_Schottky, Diode_SMD:D_SOD-123F, symbol Device:D_Schottky
- added J4: Conn_01x02_Pin, Connector_Molex:Molex_PicoBlade_53047-0210_1x02_P1.25mm_Vertical, symbol Connector:Conn_01x02_Pin
- added NT1, NT2, NT3, NT4: NetTie_2, NetTie:NetTie-2_SMD_Pad0.5mm, symbol Device:NetTie_2
- added U7: SN65HVD232, Package_SO:SOIC-8_3.9x4.9mm_P1.27mm, symbol Interface_CAN_LIN:SN65HVD232
- C1, C14, C15, C19, C20, C24, C4, C48, C52, C6, C9: RS (none) -> 247-7824
- C10, C11, C12, C17, C25, C8: RS (none) -> 814-5476
- C13, C16, C21, C22, C26, C33, C50, C7: RS (none) -> 242-7313
- C23: value 10uF -> 10uF 50V; HOUSEPART YES -> (none); MF (none) -> TDK; MPN MF-CAP-1206-10uF -> C3216X7R1H106K160AE; RS (none) -> 165-6471
- C27, C3, C30, C46, C5: RS (none) -> 103-4095
- C28, C29, C31, C32, C34, C35, C36, C37, C38, C39, C40, C41, C42, C45, C47: value 10uF 50V -> 10uF; RS (none) -> 165-6471
- C43: value 10uF 50V -> 10uF; POPULATE 1 -> (none); RS (none) -> 165-6471
- C44: value 10uF -> 10uF 50V; footprint Capacitor_SMD:C_0402_1005Metric_Pad0.74x0.62mm_HandSolder -> Capacitor_SMD:C_1206_3216Metric_Pad1.33x1.80mm_HandSolder; HOUSEPART YES -> (none); MF (none) -> TDK; MPN MF-CAP-0402-1uF -> C3216X7R1H106K160AE; RS (none) -> 165-6471
- C49: value 0.1uF -> 10nF; RS (none) -> 242-7313
- DBG1, DBG2, DRV_CS1, DRV_MISO1, DRV_MOSI1, DRV_SCK1, H2, J2, J3, M1, M2, M3, U1: now left out of the parts list
- DEBUG1: RS (none) -> 546-8811
- H1, H3, H4: footprint MountingHole:MountingHole_2.2mm_M2_ISO7380 -> nautilus:MountingHole-Plated; now left out of the parts list
- IC1: Arrow Part Number DRV8353SRTAR -> 595-DRV8353SRTAT; Mouser Part Number 595-DRV8353SRTAR -> 595-DRV8353SRTAT
- IC2: Farnell (none) -> 3132392
- J1: RS (none) -> 180-5359
- L1: RS (none) -> 246-3299
- R10, R6, R8: value 100k -> 100k 1%; HOUSEPART 1 -> (none); MF (none) -> Yageo; MPN RC0402FR-077R5L -> RC0402FR-07100KL; RS (none) -> 198-7640
- R11, R7, R9: value 5.1k -> 4.7k 1%; HOUSEPART 1 -> (none); MF (none) -> Yageo; MPN RC0402FR-077R5L -> RC0402FR-074K7L; RS (none) -> 121-277
- R12: RS (none) -> 198-7640
- R13: RS (none) -> 121-277
- R14, R18: RS (none) -> 678-4697
- R17: Mouser Part Number (none) -> 81-NCP15WB473F03RC
- RA1: value 1.0mOhm 1% 2W -> 0.5mOhm 1% 2W; MPN HCS1206FTL500 -> HCS1206FTL500
- RA2, RA3: value 1.0mOhm 1% 2W -> 0.5mOhm 1% 2W
- U4: RS (none) -> 201-8320
Connections:
- net +3.3V: now also C23.1, U7.3 (VCC); no longer C23.2, DEBUG1.5 (Pin_5)
- net DEBUG1: now also IC2.3 (PC14-OSC32_IN); no longer IC2.34 (PA12)
- net DEBUG2: now also IC2.4 (PC15-OSC32_OUT); no longer IC2.33 (PA11)
- net DRV8323_CS: now also IC2.2 (PC13); no longer IC2.4 (PC15-OSC32_OUT)
- net GNDPWR: now also C54.2, C55.2, C56.2, C57.2, NT1.1, NT2.1, NT3.1, NT4.2; no longer C17.2, C25.2, C8.2, IC1.10 (SNA), IC1.11 (SNB), IC1.20 (SNC)
- net GNDS: now also C23.2, C53.2, NT4.1, U7.2 (GND); no longer C23.1
- net LED1: now also IC2.5 (PF0-OSC_IN); no longer IC2.44 (PB6)
- net LED2: now also IC2.6 (PF1-OSC_OUT); no longer IC2.45 (PB7)
- net MOTOR_FAULT: now also IC2.44 (PB6); no longer IC2.3 (PC14-OSC32_IN)
- net MOTOR_HIZ: now also IC2.45 (PB7); no longer IC2.2 (PC13)
- net V+: now also C54.1, C55.1, C56.1, C57.1, D3.2 (A); no longer C27.1, IC3.1 (VIN), IC3.2 (EN/UVLO)
- net FCUR1: no longer names the net of C10.1, IC2.17 (PB0), R3.2
- net FCUR2: no longer names the net of C11.1, IC2.18 (PB1), R4.2
- net FCUR3: no longer names the net of C12.1, IC2.19 (PB2), R5.2
- new net: J4.1 (Pin_1), U7.7 (CANH)
- new net: J4.2 (Pin_2), U7.6 (CANL)
- new net: C27.1, C53.1, D3.1 (K), D4.1 (K), IC3.1 (VIN), IC3.2 (EN/UVLO)
- new net +5V: D4.2 (A), DEBUG1.5 (Pin_5)
- new net CAN_RX: IC2.33 (PA11), U7.4 (R)
- new net CAN_TX: IC2.34 (PA12), U7.1 (D)
- new net SXA_N: C8.2, IC1.10 (SNA), NT2.2
- new net SXB_N: C25.2, IC1.11 (SNB), NT3.2
- new net SXC_N: C17.2, IC1.20 (SNC), NT1.2
Other:
- note added: "TEMP SENSE"
- note removed: "TEMPERATURE SENSE"
- note removed: "Why is this to GNDS and not PWR GND ?"
- note removed: "nautilus v1.0"
- title: (none) -> nautilus
- moved on the sheet: C1, C10, C11, C12, C13, C14, C15, C16, C17, C18, C19, C2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

Commit message: Minor PCB update
Parts:
- added SW1: SW_Push, Button_Switch_SMD:SW_SPST_B3U-1000P, symbol Switch:SW_Push
Connections:
- net GNDS: now also SW1.1
- net NRST: now also SW1.2
Changed lines of the file:
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@@
   (junction (at 48.26 177.8) (diameter 0) (color 0 0 0 0)
   )
+  (junction (at 158.75 99.06) (diameter 0) (color 0 0 0 0)
+  )
   (junction (at 240.03 314.96) (diameter 0) (color 0 0 0 0)
   )
@@
     (stroke (width 0) (type default))
   )
-  (wire (pts (xy 160.02 99.06) (xy 167.64 99.06))
+  (wire (pts (xy 153.67 99.06) (xy 158.75 99.06))
     (stroke (width 0.1524) (type solid))
   )
@@
     (stroke (width 0) (type default))
   )
+  (wire (pts (xy 158.75 99.06) (xy 167.64 99.06))
+    (stroke (width 0.1524) (type solid))
+  )
   (wire (pts (xy 19.05 271.78) (xy 43.18 271.78))
     (stroke (width 0) (type default))
@@
     (stroke (width 0) (type default))
   )
+  (wire (pts (xy 158.75 99.06) (xy 158.75 100.33))
+    (stroke (width 0) (type default))
+  )
   (wire (pts (xy 167.64 314.96) (xy 175.26 314.96))
     (stroke (width 0.1524) (type solid))
@@
     (stroke (width 0.1524) (type solid))
   )
+  (wire (pts (xy 158.75 113.03) (xy 158.75 110.49))
+    (stroke (width 0) (type default))
+  )
   (wire (pts (xy 196.85 326.39) (xy 196.85 327.66))
     (stroke (width 0) (type default))
@@
     (stroke (width 0.1524) (type solid))
   )
-  (wire (pts (xy 167.64 107.95) (xy 167.64 109.22))
+  (wire (pts (xy 167.64 107.95) (xy 167.64 113.03))
     (stroke (width 0) (type default))
   )
@@
     (effects (font (size 1.2446 1.2446)) (justify right bottom))
   )
-  (label "NRST" (at 160.02 99.06 180) (fields_autoplaced)
+  (label "NRST" (at 153.67 99.06 180) (fields_autoplaced)
     (effects (font (size 1.2446 1.2446)) (justify right bottom))
   )
@@
     )
   )
-  (symbol (lib_id "power:GNDS") (at 167.64 109.22 0) (unit 1)
+  (symbol (lib_id "power:GNDS") (at 167.64 113.03 0) (unit 1)
     (in_bom yes) (on_board yes) (dnp no)
-    (property "Reference" "#PWR049" (at 167.64 115.57 0)
+    (property "Reference" "#PWR049" (at 167.64 119.38 0)
       (effects (font (size 1.27 1.27)) hide)
     )
-    (property "Value" "GNDS" (at 162.56 110.49 0)
+    (property "Value" "GNDS" (at 162.56 114.3 0)
       (effects (font (size 1.27 1.27)))
     )
-    (property "Footprint" "" (at 167.64 109.22 0)
+    (property "Footprint" "" (at 167.64 113.03 0)
       (effects (font (size 1.27 1.27)) hide)
     )
-    (property "Datasheet" "" (at 167.64 109.22 0)
+    (property "Datasheet" "" (at 167.64 113.03 0)
       (effects (font (size 1.27 1.27)) hide)
     )
@@
     )
   )
+  (symbol (lib_id "power:GNDS") (at 158.75 113.03 0) (unit 1)
+    (in_bom yes) (on_board yes) (dnp no)
+    (property "Reference" "#PWR062" (at 158.75 119.38 0)
+      (effects (font (size 1.27 1.27)) hide)
+    )
+    (property "Value" "GNDS" (at 153.67 114.3 0)
+      (effects (font (size 1.27 1.27)))
+    )
+    (property "Footprint" "" (at 158.75 113.03 0)
+      (effects (font (size 1.27 1.27)) hide)
+    )
+    (property "Datasheet" "" (at 158.75 113.03 0)
+      (effects (font (size 1.27 1.27)) hide)
+    )
+    (pin "1")
+    (instances
+      (project "nautilus"
+        (path "/153372ee-bcdd-4b24-a68f-0b89c1a33ebf"
+          (reference "#PWR062") (unit 1)
+        )
+      )
+    )
+  )
   (symbol (lib_id "Device:C") (at 278.13 322.58 0) (unit 1)
     (in_bom yes) (on_board yes) (dnp no)
@@
         )
       )
+    )
+  )
+  (symbol (lib_id "Switch:SW_Push") (at 158.75 105.41 90) (unit 1)
+    (in_bom yes) (on_board yes) (dnp no)
+    (property "Reference" "SW1" (at 149.86 104.14 90)
+      (effects (font (size 1.27 1.27)) (justify right))
+    )
+    (property "Value" "SW_Push" (at 147.32 106.68 90)
+      (effects (font (size 1.27 1.27)) (justify right))
+    )
+    (property "Footprint" "Button_Switch_SMD:SW_SPST_B3U-1000P" (at 153.67 105.41 0)
+      (effects (font (size 1.27 1.27)) hide)
+    )
+    (property "Datasheet" "~" (at 153.67 105.41 0)
+      (effects (font (size 1.27 1.27)) hide)
+    )
+    (pin "1")
+    (pin "2")
+    (instances
+      (project "nautilus"
+        (path "/153372ee-bcdd-4b24-a68f-0b89c1a33ebf"
+          (reference "SW1") (unit 1)
+        )
+      )

Commit message: [Hardware] First prototype order
Parts:
- C27, C30: footprint Capacitor_SMD:C_0603_1608Metric_Pad1.08x0.95mm_HandSolder -> Capacitor_SMD:C_0402_1005Metric_Pad0.74x0.62mm_HandSolder
- IC1: footprint QFN50P600X600X80-41N-D -> nautilus:QFN50P600X600X80-41N-D
- SPI1: RS 515-1541 -> 752-1807P
- SPI2: RS 515-1541 -> 515-1513
- SW1: RS (none) -> 233-4109
Changed lines of the file:
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@@
       (effects (font (size 1.27 1.27)) (justify left bottom) hide)
     )
-    (property "RS" "    515-1541" (at 68.58 76.2 0)
+    (property "RS" "    752-1807P" (at 68.58 76.2 0)
       (effects (font (size 1.27 1.27)) hide)
     )
@@
       (effects (font (size 1.016 1.016)) (justify left bottom))
     )
-    (property "Footprint" "Capacitor_SMD:C_0603_1608Metric_Pad1.08x0.95mm_HandSolder" (at 169.8752 361.95 0)
+    (property "Footprint" "Capacitor_SMD:C_0402_1005Metric_Pad0.74x0.62mm_HandSolder" (at 169.8752 361.95 0)
       (effects (font (size 1.27 1.27)) hide)
     )
@@
       (effects (font (size 1.27 1.27)) hide)
     )
+    (property "RS" "    233-4109" (at 158.75 105.41 90)
+      (effects (font (size 1.27 1.27)) hide)
+    )
     (pin "1")
     (pin "2")
@@
       (effects (font (size 1.27 1.27)))
     )
-    (property "Footprint" "QFN50P600X600X80-41N-D" (at 85.09 439.09 0)
+    (property "Footprint" "nautilus:QFN50P600X600X80-41N-D" (at 85.09 439.09 0)
       (effects (font (size 1.27 1.27)) (justify left top) hide)
     )
@@
       (effects (font (size 1.27 1.27)) (justify left bottom) hide)
     )
-    (property "RS" "    515-1541" (at 26.67 177.8 0)
+    (property "RS" "515-1513" (at 26.67 177.8 0)
       (effects (font (size 1.27 1.27)) hide)
     )
@@
       (effects (font (size 1.016 1.016)) (justify left bottom))
     )
-    (property "Footprint" "Capacitor_SMD:C_0603_1608Metric_Pad1.08x0.95mm_HandSolder" (at 180.0352 361.95 0)
-      (effects (font (size 1.27 1.27)) hide)
-    )
+    (property "Footprint" "Capacitor_SMD:C_0402_1005Metric_Pad0.74x0.62mm_HandSolder" (at 180.0352 361.95 0)
+      (effects (font (size 1.27 1.27)) hide)
+    )
