File: nautilus/hw/nautilus.kicad_sch (KiCad schematic)
At the start: 120 parts, among them IC1 DRV8353SRTAR, IC3 MAX15062AATA+T, J1 XT30XT30PW_MALE, J2 Conn_01x02_Pin, J3 Conn_01x02_Pin, J4 Conn_01x02_Pin, M1 PAD24AWG_PAD, M2 PAD24AWG_PAD, M3 PAD24AWG_PAD, SW1 SW_Push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

Commit message: Minor PCB fixup
Parts:
- added NT5: NetTie_2, NetTie:NetTie-2_SMD_Pad0.5mm, symbol Device:NetTie_2
Connections:
- net GNDPWR: now also NT5.2
- net GNDS: now also NT5.1
Changed lines of the file:
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@@
     (stroke (width 0) (type default))
   )
+  (wire (pts (xy 58.42 26.67) (xy 58.42 29.21))
+    (stroke (width 0) (type default))
+  )
   (wire (pts (xy 205.74 242.57) (xy 205.74 246.38))
     (stroke (width 0) (type default))
@@
     (stroke (width 0) (type default))
   )
+  (wire (pts (xy 45.72 26.67) (xy 49.53 26.67))
+    (stroke (width 0) (type default))
+  )
   (wire (pts (xy 22.86 350.52) (xy 22.86 355.6))
     (stroke (width 0) (type default))
@@
     (stroke (width 0) (type default))
   )
+  (wire (pts (xy 54.61 26.67) (xy 58.42 26.67))
+    (stroke (width 0) (type default))
+  )
   (wire (pts (xy 210.82 314.96) (xy 218.44 314.96))
     (stroke (width 0.1524) (type solid))
@@
     (stroke (width 0) (type default))
   )
+  (wire (pts (xy 45.72 26.67) (xy 45.72 29.21))
+    (stroke (width 0) (type default))
+  )
   (wire (pts (xy 101.6 278.13) (xy 115.57 278.13))
     (stroke (width 0) (type default))
@@
     )
   )
+  (symbol (lib_id "Device:NetTie_2") (at 52.07 26.67 180) (unit 1)
+    (in_bom no) (on_board yes) (dnp no)
+    (property "Reference" "NT5" (at 52.07 27.94 0)
+      (effects (font (size 1.27 1.27)))
+    )
+    (property "Value" "NetTie_2" (at 52.07 30.48 0)
+      (effects (font (size 1.27 1.27)))
+    )
+    (property "Footprint" "NetTie:NetTie-2_SMD_Pad0.5mm" (at 52.07 26.67 0)
+      (effects (font (size 1.27 1.27)) hide)
+    )
+    (property "Datasheet" "~" (at 52.07 26.67 0)
+      (effects (font (size 1.27 1.27)) hide)
+    )
+    (pin "1")
+    (pin "2")
+    (instances
+      (project "nautilus"
+        (path "/153372ee-bcdd-4b24-a68f-0b89c1a33ebf"
+          (reference "NT5") (unit 1)
+        )
+      )
+    )
+  )
   (symbol (lib_id "Device:C") (at 173.99 99.06 0) (unit 1)
     (in_bom yes) (on_board yes) (dnp no)
@@
     )
   )
+  (symbol (lib_id "power:GNDPWR") (at 45.72 29.21 0) (unit 1)
+    (in_bom yes) (on_board yes) (dnp no) (fields_autoplaced)
+    (property "Reference" "#PWR034" (at 45.72 34.29 0)
+      (effects (font (size 1.27 1.27)) hide)
+    )
+    (property "Value" "GNDPWR" (at 45.593 33.02 0)
+      (effects (font (size 1.27 1.27)))
+    )
+    (property "Footprint" "" (at 45.72 30.48 0)
+      (effects (font (size 1.27 1.27)) hide)
+    )
+    (property "Datasheet" "" (at 45.72 30.48 0)
+      (effects (font (size 1.27 1.27)) hide)
+    )
+    (pin "1")
+    (instances
+      (project "nautilus"
+        (path "/153372ee-bcdd-4b24-a68f-0b89c1a33ebf"
+          (reference "#PWR034") (unit 1)
+        )
+      )
+    )
+  )
   (symbol (lib_id "Device:C") (at 156.21 358.14 0) (unit 1)
     (in_bom yes) (on_board yes) (dnp no)
@@
         )
       )
+    )
+  )
+  (symbol (lib_id "power:GNDS") (at 58.42 29.21 0) (unit 1)
+    (in_bom yes) (on_board yes) (dnp no) (fields_autoplaced)
+    (property "Reference" "#PWR038" (at 58.42 35.56 0)
+      (effects (font (size 1.27 1.27)) hide)
+    )
+    (property "Value" "GNDS" (at 58.42 34.29 0)
+      (effects (font (size 1.27 1.27)))
+    )
+    (property "Footprint" "" (at 58.42 29.21 0)
+      (effects (font (size 1.27 1.27)) hide)
+    )
+    (property "Datasheet" "" (at 58.42 29.21 0)
+      (effects (font (size 1.27 1.27)) hide)
+    )
+    (pin "1")
+    (instances
+      (project "nautilus"
+        (path "/153372ee-bcdd-4b24-a68f-0b89c1a33ebf"
+          (reference "#PWR038") (unit 1)
+        )
+      )

Commit message: Add missing build files. Update resistor value for led brightness.
Parts:
- R15: value 2k -> 5.1k
Changed lines of the file:
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@@
       (effects (font (size 1.016 1.016)) (justify left top))
     )
-    (property "Value" "2k" (at 121.92 131.064 0)
+    (property "Value" "5.1k" (at 121.92 131.064 0)
       (effects (font (size 1.016 1.016)) (justify left bottom))
     )

Commit message: Update current sense filtering to 14kHz to avoid aliasing.
Parts:
- C10, C11, C12: value 1000pF -> 1uF
- D3, D4: Mouser Part Number 833-SS24FL-TP -> 833-SMD210PLQ-TP
- L1: Mouser (none) -> SRN4018
- R3, R4, R5: value 22 -> 68
- RA1, RA2, RA3: Mouser (none) -> 504-MSMA2512R0005FGM
