File: nautilus/hw/nautilus.kicad_pcb (KiCad board)
At the start: 4 copper layers, 54.7 x 55 mm, 120 parts, among them IC1 DRV8353SRTAR, IC3 MAX15062AATA+T, J1 XT30XT30PW_MALE, J2 Conn_01x02_Pin, J3 Conn_01x02_Pin, J4 Conn_01x02_Pin, M1 PAD24AWG_PAD, M2 PAD24AWG_PAD, M3 PAD24AWG_PAD, SW1 SW_Push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

Commit message: [Hardware] V2 board order
Parts:
- moved C48 1.50 mm to (161.2, 68.4)
- moved R15 1.50 mm to (159.1, 68.4)
- moved R16 1.50 mm to (160.2, 68.4)
- moved M1 0.10 mm to (151.2, 92.3)
- moved R10 0.07 mm to (125.0, 83.3)
Routing:
- net Net-(D1-A): track 17.2 -> 18.8 mm
- net Net-(D2-A): track 16.2 -> 17.7 mm
- net Net-(J4-Pin_2): track 6.35 -> 7.13 mm
- net Net-(J4-Pin_1): track 4.56 -> 5.09 mm
Other:
- board text added: "GND"
- board text added: "TX"

Commit message: Minor PCB fixup
Parts:
- added NT5: NetTie_2, NetTie:NetTie-2_SMD_Pad0.5mm, B.Cu at (137.7, 65.8)
- moved NT4 4.25 mm to (137.7, 71.2)
Routing:
- net GNDPWR: track 8.72 -> 12.3 mm
- net GNDS: track 7.23 -> 4.43 mm, vias 58 -> 55
Changed lines of the file:
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@@
     (property "ki_keywords" "cap capacitor")
     (attr smd)
-    (fp_text reference "C4" (at 1.6325 0.4) (layer "F.SilkS")
+    (fp_text reference "C4" (at 1.7525 0.4) (layer "F.SilkS")
         (effects (font (size 1 1) (thickness 0.15)))
     )
@@
   )
   (footprint "NetTie:NetTie-2_SMD_Pad0.5mm" (layer "B.Cu")
-    (at 135.4 67.6 90)
+    (at 137.65 65.8 -90)
     (descr "Net tie, 2 pin, 0.5mm square SMD pads")
     (tags "net tie")
@@
     (attr exclude_from_pos_files exclude_from_bom)
     (net_tie_pad_groups "1, 2")
-    (fp_text reference "NT4" (at 0 1.2 90) (layer "B.SilkS") hide
+    (fp_text reference "NT5" (at 0 1.2 90) (layer "B.SilkS") hide
         (effects (font (size 1 1) (thickness 0.15)) (justify mirror))
     )
@@
       )
       (stroke (width 0) (type solid)) (fill solid) (layer "B.Cu"))
+    (pad "1" smd circle (at -0.5 0 270) (size 0.5 0.5) (layers "B.Cu")
+      (net 88 "GNDS") (pinfunction "1") (pintype "passive"))
+    (pad "2" smd circle (at 0.5 0 270) (size 0.5 0.5) (layers "B.Cu")
+      (net 87 "GNDPWR") (pinfunction "2") (pintype "passive"))
+  )
+  (footprint "NetTie:NetTie-2_SMD_Pad0.5mm" (layer "B.Cu")
+    (at 137.65 71.2 90)
+    (descr "Net tie, 2 pin, 0.5mm square SMD pads")
+    (tags "net tie")
+    (property "Sheetfile" "nautilus.kicad_sch")
+    (property "Sheetname" "")
+    (property "exclude_from_bom" "")
+    (property "ki_description" "Net tie, 2 pins")
+    (property "ki_keywords" "net tie short")
+    (attr exclude_from_pos_files exclude_from_bom)
+    (net_tie_pad_groups "1, 2")
+    (fp_text reference "NT4" (at 0 1.2 270) (layer "B.SilkS") hide
+        (effects (font (size 1 1) (thickness 0.15)) (justify mirror))
+    )
+    (fp_text value "NetTie_2" (at 0 -1.2 270) (layer "B.Fab") hide
+        (effects (font (size 1 1) (thickness 0.15)) (justify mirror))
+    )
+    (fp_poly
+      (pts
+        (xy -0.5 0.25)
+        (xy 0.5 0.25)
+        (xy 0.5 -0.25)
+        (xy -0.5 -0.25)
+      )
+      (stroke (width 0) (type solid)) (fill solid) (layer "B.Cu"))
     (pad "1" smd circle (at -0.5 0 90) (size 0.5 0.5) (layers "B.Cu")
       (net 88 "GNDS") (pinfunction "1") (pintype "passive"))
@@
       (net 87 "GNDPWR") (pinfunction "1") (pintype "passive"))
     (pad "2" thru_hole circle (at -5 0 180) (size 3.5 3.5) (drill 1.9) (layers "*.Cu" "*.Mask")
-      (net 5 "V+") (pinfunction "2") (pintype "passive"))
+      (net 5 "V+") (pinfunction "2") (pintype "passive") (thermal_bridge_width 1))
     (model "${KICAD6_3DMODEL_DIR}/Connector_AMASS.3dshapes/AMASS_XT30PW-M_1x02_P2.50mm_Horizontal.wrl"
       (offset (xyz 0 0 0))
@@
   (segment (start 158.201 84.906026) (end 154.594974 81.3) (width 0.25) (layer "B.Cu") (net 28))
   (segment (start 150.7 81.3) (end 150.5 81.1) (width 0.25) (layer "B.Cu") (net 28))
+  (segment (start 162.087191 93.75) (end 162.297191 93.96) (width 0.25) (layer "F.Cu") (net 29))
+  (segment (start 161.130874 93.75) (end 162.087191 93.75) (width 0.25) (layer "F.Cu") (net 29))
+  (segment (start 161.127361 93.746487) (end 161.130874 93.75) (width 0.25) (layer "F.Cu") (net 29))
   (segment (start 162.297191 93.96) (end 163.13 93.96) (width 0.25) (layer "F.Cu") (net 29))
-  (segment (start 161.127361 93.746487) (end 161.251861 93.621987) (width 0.25) (layer "F.Cu") (net 29))
-  (segment (start 161.959178 93.621987) (end 162.297191 93.96) (width 0.25) (layer "F.Cu") (net 29))
-  (segment (start 161.251861 93.621987) (end 161.959178 93.621987) (width 0.25) (layer "F.Cu") (net 29))
   (via (at 161.127361 93.746487) (size 0.5) (drill 0.2) (layers "F.Cu" "B.Cu") (net 29))
   (segment (start 157.851 88.006026) (end 157.851 85.051) (width 0.25) (layer "B.Cu") (net 29))
@@
   (segment (start 145.7 86.6) (end 145.7 86.05) (width 0.25) (layer "F.Cu") (net 64))
   (segment (start 146.9 87.3) (end 148.22 87.3) (width 0.25) (layer "F.Cu") (net 65))
-  (segment (start 160.21 77.4) (end 159.41 78.2) (width 0.25) (layer "F.Cu") (net 66))
-  (segment (start 161.7 77.4) (end 160.21 77.4) (width 0.25) (layer "F.Cu") (net 66))
+  (segment (start 161.7 77.4) (end 160.3 77.4) (width 0.25) (layer "F.Cu") (net 66))
+  (segment (start 159.4 78.3) (end 159.4 78.665) (width 0.25) (layer "F.Cu") (net 66))
+  (segment (start 160.3 77.4) (end 159.4 78.3) (width 0.25) (layer "F.Cu") (net 66))
   (via (at 159.1 67.805) (size 0.5) (drill 0.2) (layers "F.Cu" "B.Cu") (net 67))
   (via (at 146.95 56.1) (size 0.5) (drill 0.2) (layers "F.Cu" "B.Cu") (net 67))
@@
   (via (at 154.34 78.02) (size 0.5) (drill 0.2) (layers "F.Cu" "B.Cu") (net 87))
   (via (at 134.4 90.6) (size 0.5) (drill 0.2) (layers "F.Cu" "B.Cu") (net 87))
-  (segment (start 135.4 67.1) (end 136.25 67.1) (width 0.5) (layer "B.Cu") (net 87))
+  (segment (start 137.65 68.5) (end 137.65 66.3) (width 0.5) (layer "B.Cu") (net 87))
+  (segment (start 137.65 70.7) (end 137.65 68.5) (width 0.5) (layer "B.Cu") (net 87))
   (segment (start 143.7 92.5) (end 143.7 93.15) (width 0.25) (layer "F.Cu") (net 88))
   (segment (start 154.2255 62.3805) (end 154.2255 60.4495) (width 0.25) (layer "F.Cu") (net 88))
@@
   (via (at 157.985 101) (size 0.5) (drill 0.2) (layers "F.Cu" "B.Cu") (net 88))
   (via (at 162.2375 72.475) (size 0.5) (drill 0.2) (layers "F.Cu" "B.Cu") (net 88))
-  (via (at 135.4 68.9) (size 0.7) (drill 0.3) (layers "F.Cu" "B.Cu") (net 88))
   (via (at 160.895 82.8) (size 0.5) (drill 0.2) (layers "F.Cu" "B.Cu") (net 88))
   (via (at 145.4 95.3) (size 0.5) (drill 0.2) (layers "F.Cu" "B.Cu") (net 88))
@@
   (via (at 163.13 90.46) (size 0.5) (drill 0.2) (layers "F.Cu" "B.Cu") (net 88))
   (via (at 157.985 100.029) (size 0.5) (drill 0.2) (layers "F.Cu" "B.Cu") (net 88))
-  (via (at 135.4 69.8) (size 0.7) (drill 0.3) (layers "F.Cu" "B.Cu") (net 88))
   (via (at 152 107.4) (size 0.5) (drill 0.2) (layers "F.Cu" "B.Cu") (net 88))
   (via (at 166.1 81.225) (size 0.5) (drill 0.2) (layers "F.Cu" "B.Cu") (net 88))
@@
   (via (at 142.2 87.8) (size 0.5) (drill 0.2) (layers "F.Cu" "B.Cu") (net 88))
   (via (at 158.9 75.07) (size 0.5) (drill 0.2) (layers "F.Cu" "B.Cu") (net 88))
-  (via (at 134.3 69.8) (size 0.7) (drill 0.3) (layers "F.Cu" "B.Cu") (net 88))
   (via (at 154.2255 62.3805) (size 0.5) (drill 0.2) (layers "F.Cu" "B.Cu") (net 88))
   (via (at 144.4 91.2) (size 0.5) (drill 0.2) (layers "F.Cu" "B.Cu") (net 88))
@@
   (via (at 143.2 91.2) (size 0.5) (drill 0.2) (layers "F.Cu" "B.Cu") (net 88))
   (via (at 142.2 90.2) (size 0.5) (drill 0.2) (layers "F.Cu" "B.Cu") (net 88))
-  (segment (start 135.4 68.9) (end 135.4 69.8) (width 0.5) (layer "B.Cu") (net 88))
-  (segment (start 135.4 68.9) (end 135.4 68.1) (width 0.5) (layer "B.Cu") (net 88))
-  (segment (start 135.4 69.8) (end 134.3 69.8) (width 0.5) (layer "B.Cu") (net 88))
   (segment (start 131.4975 89.897) (end 131.4975 89.1) (width 0.25) (layer "F.Cu") (net 89))
   (segment (start 161.79 79.7) (end 160.9 79.7) (width 0.25) (layer "F.Cu") (net 89))
@@
     (polygon
       (pts
-        (xy 155.4 57.8)
+        (xy 155.4 57.9)
         (xy 139 57.9)
-        (xy 139 62.5)
-        (xy 155.1 62.4)
-        (xy 155.2 74)
-        (xy 158.75 73.95)
-        (xy 158.8 83.5)
-        (xy 153.5 83.5)
-        (xy 153.5 92)
-        (xy 141.675 92)
-        (xy 141.7 110.6)
-        (xy 175.8 110.6)
-        (xy 175.7 57.7)
+        (xy 139 62.6)
+        (xy 155.1 62.6)
+        (xy 155.1 74.1)
+        (xy 158.8 74.1)
+        (xy 158.8 83.6)
+        (xy 153.5 83.6)
+        (xy 153.5 92.1)
+        (xy 141.675 92.1)
+        (xy 141.7 110.7)
+        (xy 175.8 110.7)
+        (xy 175.7 57.8)
       )
     )
@@
     (polygon
       (pts
-        (xy 152.8 63.8)
-        (xy 152.6 70.32)
-        (xy 152.6 70.3)
-        (xy 152.8 78.3)
-        (xy 158.1 78.3)
-        (xy 158.1 82.6)
-        (xy 152.6 82.6)
-        (xy 152.6 86.1)
-        (xy 147.697069 86.1)
-        (xy 147.7 92.9)
-        (xy 140.5 93)
-        (xy 140.5 109)
-        (xy 122.1 109.1)
-        (xy 122.1 63.8)
+        (xy 153 63.8)
+        (xy 153 78.15)
+        (xy 158.1 78.15)
+        (xy 158.1 82.45)
+        (xy 152.6 82.45)
+        (xy 152.6 85.95)
+        (xy 147.697069 85.95)
+        (xy 147.7 92.75)
+        (xy 140.5 92.85)
+        (xy 140.5 108.85)
+        (xy 122.1 108.95)
+        (xy 122.1 63.85)
       )
     )
@@
     (connect_pads (clearance 0.15))
     (min_thickness 0.15) (filled_areas_thickness no)
-    (fill yes (thermal_gap 0.2) (thermal_bridge_width 0.3))
+    (fill yes (thermal_gap 0.2) (thermal_bridge_width 1))
     (polygon
       (pts

Commit message: Update current sense filtering to 14kHz to avoid aliasing.
Parts:
- C10, C11, C12: value 1000pF -> 1uF
- R15: value 2k -> 5.1k
- R3, R4, R5: value 22 -> 68
- renumbered locked to U6
